Commit message: added meshes for robotiq 2f85 gripper

File: kinova_gym/models/urdf/gen3_robotiq_2f_85.urdf (robot description, URDF)
Before this commit: robot gen3_robotiq_2f_85, 24 links, 23 joints
Links:
- link base_link: geometry collision mesh filename=meshes/base_link.STL; visual mesh filename=meshes/base_link.STL
- link bracelet_link: geometry collision mesh filename=meshes/bracelet_with_vision_link.STL; visual mesh filename=meshes/bracelet_with_vision_link.STL
- link forearm_link: geometry collision mesh filename=meshes/forearm_link.STL; visual mesh filename=meshes/forearm_link.STL
- link half_arm_1_link: geometry collision mesh filename=meshes/half_arm_1_link.STL; visual mesh filename=meshes/half_arm_1_link.STL
- link half_arm_2_link: geometry collision mesh filename=meshes/half_arm_2_link.STL; visual mesh filename=meshes/half_arm_2_link.STL
- link left_inner_finger: geometry collision mesh filename=meshes/robotiq_2f_85/meshes/collision/robotiq_arg2f_85_inne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 scale=0.001 0.001 0.001; visual mesh filename=meshes/robotiq_2f_85/meshes/visual/robotiq_arg2f_85_inner_f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 scale=0.001 0.001 0.001
- link left_inner_knuckle: geometry collision mesh filename=meshes/robotiq_2f_85/meshes/collision/robotiq_arg2f_85_inne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 scale=0.001 0.001 0.001; visual mesh filename=meshes/robotiq_2f_85/meshes/visual/robotiq_arg2f_85_inner_k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 scale=0.001 0.001 0.001
- link left_outer_finger: geometry collision mesh filename=meshes/robotiq_2f_85/meshes/collision/robotiq_arg2f_85_oute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 scale=0.001 0.001 0.001; visual mesh filename=meshes/robotiq_2f_85/meshes/visual/robotiq_arg2f_85_outer_f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 scale=0.001 0.001 0.001
- link left_outer_knuckle: geometry collision mesh filename=meshes/robotiq_2f_85/meshes/collision/robotiq_arg2f_85_oute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 scale=0.001 0.001 0.001; visual mesh filename=meshes/robotiq_2f_85/meshes/visual/robotiq_arg2f_85_outer_k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 scale=0.001 0.001 0.001
- link right_inner_finger: geometry collision mesh filename=meshes/robotiq_2f_85/meshes/collision/robotiq_arg2f_85_inne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 scale=0.001 0.001 0.001; visual mesh filename=meshes/robotiq_2f_85/meshes/visual/robotiq_arg2f_85_inner_f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 scale=0.001 0.001 0.001
- link right_inner_knuckle: geometry collision mesh filename=meshes/robotiq_2f_85/meshes/collision/robotiq_arg2f_85_inne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 scale=0.001 0.001 0.001; visual mesh filename=meshes/robotiq_2f_85/meshes/visual/robotiq_arg2f_85_inner_k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 scale=0.001 0.001 0.001
- link right_outer_finger: geometry collision mesh filename=meshes/robotiq_2f_85/meshes/collision/robotiq_arg2f_85_oute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 scale=0.001 0.001 0.001; visual mesh filename=meshes/robotiq_2f_85/meshes/visual/robotiq_arg2f_85_outer_f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 scale=0.001 0.001 0.001
- link right_outer_knuckle: geometry collision mesh filename=meshes/robotiq_2f_85/meshes/collision/robotiq_arg2f_85_oute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 scale=0.001 0.001 0.001; visual mesh filename=meshes/robotiq_2f_85/meshes/visual/robotiq_arg2f_85_outer_k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 scale=0.001 0.001 0.001
- link robotiq_arg2f_base_link: geometry collision mesh filename=meshes/robotiq_2f_85/meshes/collision/robotiq_arg2f_base_li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; visual mesh filename=meshes/robotiq_2f_85/meshes/collision/robotiq_arg2f_base_li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
- link shoulder_link: geometry collision mesh filename=meshes/shoulder_link.STL; visual mesh filename=meshes/shoulder_link.STL
- link spherical_wrist_1_link: geometry collision mesh filename=meshes/spherical_wrist_1_link.STL; visual mesh filename=meshes/spherical_wrist_1_link.STL
- link spherical_wrist_2_link: geometry collision mesh filename=meshes/spherical_wrist_2_link.STL; visual mesh filename=meshes/spherical_wrist_2_link.STL
