Commit message: added test script to load kinova in pb

File: kinova_gym/models/urdf/gen3.urdf (robot description, URDF)
Before this commit: robot gen3_robotiq_2f_85, 14 links, 13 joints
Links:
- link base_link: geometry collision mesh filename=meshes/base_link.STL; visual mesh filename=meshes/base_link.STL
- link bracelet_link: geometry collision mesh filename=meshes/bracelet_with_vision_link.STL; visual mesh filename=meshes/bracelet_with_vision_link.STL
- link forearm_link: geometry collision mesh filename=meshes/forearm_link.STL; visual mesh filename=meshes/forearm_link.STL
- link half_arm_1_link: geometry collision mesh filename=meshes/half_arm_1_link.STL; visual mesh filename=meshes/half_arm_1_link.STL
- link half_arm_2_link: geometry collision mesh filename=meshes/half_arm_2_link.STL; visual mesh filename=meshes/half_arm_2_link.STL
- link shoulder_link: geometry collision mesh filename=meshes/shoulder_link.STL; visual mesh filename=meshes/shoulder_link.STL
- link spherical_wrist_1_link: geometry collision mesh filename=meshes/spherical_wrist_1_link.STL; visual mesh filename=meshes/spherical_wrist_1_link.STL
- link spherical_wrist_2_link: geometry collision mesh filename=meshes/spherical_wrist_2_link.STL; visual mesh filename=meshes/spherical_wrist_2_link.STL

Commit message: added script to load robot in mujoco

File: kinova_gym/models/urdf/gen3.urdf (robot description, URDF)
Before this commit: robot gen3_robotiq_2f_85, 14 links, 13 joints
Links:
- removed link table
Joints:
- removed joint arm_table_joint
